Commit message: Update

File: my_robot/urdf/my_robot.xacro (robot description, xacro)
@@ -67,5 +67,4 @@
         <box size=".4 .2 .1"/>
       </geometry>
-			<material name="black"/>
     </visual>
     <collision name='back_caster_collision'>
@@ -190,3 +189,12 @@
     </collision>
   </link>
+	<gazebo reference="left_wheel">
+		<material>Gazebo/Red</material>
+	</gazebo>
+	<gazebo reference="right_wheel">
+		<material>Gazebo/Red</material>
+	</gazebo>
+	<gazebo reference="chassis">
+		<material>Gazebo/Black</material>
+	</gazebo>
 </robot>
